File: alarmclock3.sch (EAGLE design)
At the start: 28 parts, among them X1 MKDSN1,5/2-5,08, X2 MKDSN1,5/2-5,08

Commit message: - separate gnd from 18v stage and 3.3v stage - add 2 gpio as terminal block (2 external push button) - complete the bom
Parts:
- removed C1: (no value), SparkFun-Passives:CAP_POLPTH3
- added C11: 330uF/25V, SparkFun-Passives:CAP_POLPTH2
- added R4, R6: 10k, SparkFun-Passives:RESISTOR0603-RES
- added X3, X4: MKDSN1,5/2-5,08, con-phoenix-508:MKDSN1,5/2-5,08
Connections:
- new net +3V3: R1.2, R4.2, R6.2, U$3.!RESET!, U$3.AVDD, U$3.DVDD, U$5.VCC-3.3V
- new net +5V: U$5.VCC-5V, U$5.VCC-5VB
- new net N$29: C11.-, U$2.VO-, U$4.GND
- net GND: now also X3-2.KL, X4-2.KL; no longer C1.-, U$2.VO-, U$4.GND
- net N$3: now also C11.+; no longer C1.+
- net N$6: now also R6.1, U$5.IO3, X4-1.KL; no longer R1.2, U$3.AVDD, U$3.DVDD, U$5.VCC-3.3V
- net N$8: now also R4.1, U$5.IO2, X3-1.KL; no longer U$3.!RESET!, U$5.VCC-5V, U$5.VCC-5VB
Other:
- moved on the sheet: R1

Commit message: add extension to the skywriter (https://www.modmypi.com/raspberry-pi/breakout-boards/pimoroni/pimoroni-skywriter)
Parts:
- added U$10: SKYWRITER, skywriter:SKYWRITER
Connections:
- new net N$30: U$10.SDA, U$5.TWI2-SDA
- new net N$31: U$10.SCL, U$5.TWI2-CLK
- new net N$32: U$10.RESET, U$5.IO1
- new net N$33: U$10.TRFR, U$5.IO0
- net +3V3: now also U$10.VCC3.3
- net GND: now also U$10.GND
Changed lines of the file:
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@@
 <part name="+3V5" library="supply1" deviceset="+3V3" device=""/>
 <part name="+3V6" library="supply1" deviceset="+3V3" device=""/>
+<part name="U$10" library="skywriter" deviceset="SKYWRITER" device=""/>
+<part name="+3V7" library="supply1" deviceset="+3V3" device=""/>
+<part name="SUPPLY29" library="supply2" deviceset="GND" device=""/>
 </parts>
 <sheets>
@@
 <instance part="+3V5" gate="G$1" x="-63.5" y="5.08"/>
 <instance part="+3V6" gate="G$1" x="-63.5" y="-30.48"/>
+<instance part="U$10" gate="G$1" x="-71.12" y="38.1" rot="R180"/>
+<instance part="+3V7" gate="G$1" x="-60.96" y="53.34"/>
+<instance part="SUPPLY29" gate="GND" x="-60.96" y="22.86"/>
 </instances>
 <busses>
@@
 <pinref part="SUPPLY28" gate="GND" pin="GND"/>
 <wire x1="-71.12" y1="-48.26" x2="-63.5" y2="-48.26" width="0.1524" layer="91"/>
+</segment>
+<segment>
+<pinref part="U$10" gate="G$1" pin="GND"/>
+<pinref part="SUPPLY29" gate="GND" pin="GND"/>
 </segment>
 </net>
@@
 <pinref part="+3V5" gate="G$1" pin="+3V3"/>
 </segment>
+<segment>
+<pinref part="U$10" gate="G$1" pin="VCC3.3"/>
+<pinref part="+3V7" gate="G$1" pin="+3V3"/>
+</segment>
 </net>
 <net name="N$6" class="0">
@@
 </segment>
 </net>
+<net name="N$30" class="0">
+<segment>
+<pinref part="U$5" gate="G$1" pin="TWI2-SDA"/>
+<wire x1="-20.32" y1="12.7" x2="-40.64" y2="12.7" width="0.1524" layer="91"/>
+<wire x1="-40.64" y1="12.7" x2="-40.64" y2="45.72" width="0.1524" layer="91"/>
+<pinref part="U$10" gate="G$1" pin="SDA"/>
+<wire x1="-40.64" y1="45.72" x2="-60.96" y2="45.72" width="0.1524" layer="91"/>
+</segment>
+</net>
+<net name="N$31" class="0">
+<segment>
+<pinref part="U$5" gate="G$1" pin="TWI2-CLK"/>
+<wire x1="-20.32" y1="7.62" x2="-43.18" y2="7.62" width="0.1524" layer="91"/>
+<wire x1="-43.18" y1="7.62" x2="-43.18" y2="40.64" width="0.1524" layer="91"/>
+<pinref part="U$10" gate="G$1" pin="SCL"/>
+<wire x1="-43.18" y1="40.64" x2="-60.96" y2="40.64" width="0.1524" layer="91"/>
+</segment>
+</net>
+<net name="N$32" class="0">
+<segment>
+<pinref part="U$5" gate="G$1" pin="IO1"/>
+<wire x1="-20.32" y1="2.54" x2="-45.72" y2="2.54" width="0.1524" layer="91"/>
+<wire x1="-45.72" y1="2.54" x2="-45.72" y2="35.56" width="0.1524" layer="91"/>
+<pinref part="U$10" gate="G$1" pin="RESET"/>
+<wire x1="-45.72" y1="35.56" x2="-60.96" y2="35.56" width="0.1524" layer="91"/>
+</segment>
+</net>
+<net name="N$33" class="0">
+<segment>
+<pinref part="U$5" gate="G$1" pin="IO0"/>
+<wire x1="-20.32" y1="-7.62" x2="-48.26" y2="-7.62" width="0.1524" layer="91"/>
+<wire x1="-48.26" y1="-7.62" x2="-48.26" y2="30.48" width="0.1524" layer="91"/>
+<pinref part="U$10" gate="G$1" pin="TRFR"/>
+<wire x1="-48.26" y1="30.48" x2="-60.96" y2="30.48" width="0.1524" layer="91"/>
+</segment>
+</net>
